Commit message: Inertia fix

File: ur_description/urdf/ur10.urdf.xacro (robot description, xacro)
@@ -299,8 +299,20 @@
         </geometry>
       </collision>
+      <inertial>
+        <mass value="1e-5" />
+        <origin xyz="0 0 0" rpy="0 0 0"/>
+        <inertia ixx="1e-6" ixy="0" ixz="0" iyy="1e-6" iyz="0" izz="1e-6" />
+      </inertial>
+    </link>
+    <link name="${prefix}wrist_3_link_inertia">
       <xacro:cylinder_inertial radius="0.045" length="0.0305" mass="${wrist_3_mass}">
-        <origin xyz="0.0 ${wrist_3_length - 0.0305/2} 0.0" rpy="${pi/2} 0 0" />
-      </xacro:cylinder_inertial>
-    </link>
+        <origin xyz="0.0 0.0 0.0" rpy="0 0 0" />
+      </xacro:cylinder_inertial>
+    </link>
+    <joint name="${prefix}wrist_3_link_to_inertia" type="fixed">
+      <parent link="${prefix}wrist_3_link" />
+      <child link = "${prefix}wrist_3_link_inertia" />
+      <origin xyz="0.0 ${wrist_3_length - 0.0305/2} 0.0" rpy="${pi/2} 0 0" />
+    </joint>
     <joint name="${prefix}ee_fixed_joint" type="fixed">
       <parent link="${prefix}wrist_3_link" />
